File: OpenRX-Lite/OpenRX-Lite.kicad_sch (KiCad schematic)
At the start: 0 parts

Commit message: Consolidate docs: 1 README + KICAD_WORKFLOW + 1 DESIGN.md per receiver
- Merge SCHEMATIC.md + BOM.md into single DESIGN.md per receiver
- Delete OPENRX_ELRS_4_RECEIVER_PORTFOLIO.md (content integrated)
- Delete REPO_AUDIT_2026-03-23.md (issues addressed)
- Fold CORE_BOM into README.md architecture table
- Rename KICAD_WORKFLOW_AND_ELRS_COMPATIBILITY.md to KICAD_WORKFLOW.md
- Rewrite KICAD_WORKFLOW with step-by-step capture instructions
- Add shared libs and starter shared sheet from audit agent
Other:
- added sheet ESP32-C3 + SX1281 Core (../shared/sheets/esp32c3_sx1281_rx_core.kicad_sch)
Changed lines of the file:
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@@
 (kicad_sch
   (version 20231120)
-  (generator "eeschema")
-  (generator_version "9.0")
+  (generator "codex")
+  (generator_version "1.0")
   (paper "A3")
-  (symbol_instances)
+  (sheet
+    (at 25.4 25.4 0)
+    (size 177.8 114.3)
+    (stroke
+      (width 0)
+      (type default)
+      (color 0 0 0 0)
+    )
+    (fill
+      (color 0 0 0 0.0000)
+    )
+    (property "Sheetname" "ESP32-C3 + SX1281 Core"
+      (at 27.94 22.86 0)
+      (effects
+        (font
+          (size 1.27 1.27)
+        )
+      )
+    )
+    (property "Sheetfile" "../shared/sheets/esp32c3_sx1281_rx_core.kicad_sch"
+      (at 27.94 141.478 0)
+      (effects
+        (font
+          (size 1.27 1.27)
+        )
+        (hide yes)
+      )
+    )
+    (instances
+      (project "OpenRX-Lite"
+        (path "/8521861a-4fab-458b-8289-5e2efb91d906/d4225140-81df-42e7-abd7-e679e5ab5187"
+          (page "2")
+        )
+      )
+    )
+  )
+  (sheet_instances
+    (path "/"
+      (page "1")
+    )
+    (path "/8521861a-4fab-458b-8289-5e2efb91d906/d4225140-81df-42e7-abd7-e679e5ab5187"
+      (page "2")
+    )
+  )
 )
