File: OpenRX-Lite/esp32c3_sx1281_lite.kicad_sch (KiCad schematic)
At the start: 38 parts, among them U1 ESP32-C3FH4, U2 TLV75533PDQNR, U3 SX1281IMLTRT, X1 CJ17-400001010B20

Commit message: Update schematics: Mono RF rewiring, SKY13414 port mapping, shared libs
Mono: disconnect IPD TX_LP (unused by ELRS), route TX_HP→RF3, RX→RF1,
RFX2401C ANT→RF4. Matches BetaFPV SuperX topology.

Co-Authored-By: Claude Opus 4.6 (1M context) <noreply@anthropic.com>
Parts:
- removed USB1: DEA102700LT-6307A2, OpenRX-Shared:FILTER-SMD_4P-L1.0-W0.5-L_DEA102700LT-XXX, symbol OpenRX-Shared:DEA102700LT-6307A2
- added FL1: 2450FM07D0034T, OpenRX-Shared:FILTER-SMD_4P-L1.0-W0.5-L, symbol OpenRX-Shared:2450FM07D0034T
- added TP5: GND, OpenRX-Shared:SolderPad_1.2x2.0mm, symbol Connector:TestPoint
- AE2: now fitted
- renumbered C6 to C1, C9 to C10, C4 to C11, C5 to C12, C17 to C14, C10 to C15, C11 to C16, C15 to C17, C14 to C18, C18 to C19, C8 to C2, C16 to C20, C7 to C3, C19 to C4, C1 to C5, C2 to C6, C20 to C7, C12 to C8, C3 to C9, L to L1, R4 to R2, R2 to R3, R3 to R4
Connections:
- net CHIP_BOOT: now also TP5.1
- net GND: now also FL1.2 (GND), FL1.4 (GND)
- net at U3.22 (RFIO): now also FL1.1 (IN)
- net at AE2.3: now also FL1.3 (OUT)
