File: shared/sheets/esp32c3_sx1281_rx_core.kicad_sch (KiCad schematic)
At the start: 3 parts, among them U1 ESP32-C3FH4, X1 CJ17-400001010B20

Commit message: Unify library tables, import RFX2401C, Lite schematic capture
- All 6 projects now share OpenRX-Shared + OpenRX-Lite lib tables
- Import RFX2401C (C19213) into shared library with 3D model path fix
- OpenRX-Lite schematic: 0 ERC errors (captured in KiCad GUI)
- Add .gitignore for .lck and .history files
Parts:
- added AE2: 47948-0001, OpenRX-Shared:ANT-SMD_47948-0001, symbol OpenRX-Shared:47948-0001
- added C1, C13, C14, C15, C17, C2, C3, C4, C5: 100nF, Capacitor_SMD:C_0201_0603Metric, symbol Device:C
- added C10, C19, C8, C9: 1uF, Capacitor_SMD:C_0201_0603Metric, symbol Device:C
- added C11, C12: 10uF, Capacitor_SMD:C_0201_0603Metric, symbol Device:C
- added C16: 470nF, Capacitor_SMD:C_0201_0603Metric, symbol Device:C
- added C18: 1nF, Capacitor_SMD:C_0201_0603Metric, symbol Device:C
- added C6, C7: 10pF, Capacitor_SMD:C_0201_0603Metric, symbol Device:C
- added D1: XL-1010RGBC-WS2812B, OpenRX-Shared:LED-SMD_4P-L1.0-W1.0-TL_XL-1010RGBC-WS2812B, symbol OpenRX-Shared:XL-1010RGBC-WS2812B
- added OSC1: OW7EL89CENUNFAYLC-52M, OpenRX-Shared:OSC-SMD_4P-L2.0-W1.6-BL_TXC_7Z, symbol OpenRX-Shared:OW7EL89CENUNFAYLC-52M
- added R1, R2, R3, R4: 10k, Resistor_SMD:R_0201_0603Metric, symbol Device:R
- added TP1: RX, OpenRX-Shared:SolderPad_1.0x1.5mm, symbol Connector:TestPoint
- added TP2: TX, OpenRX-Shared:SolderPad_1.0x1.5mm, symbol Connector:TestPoint
- added TP3: 5V, OpenRX-Shared:SolderPad_1.0x1.5mm, symbol Connector:TestPoint
- added TP4: GND, OpenRX-Shared:SolderPad_1.0x1.5mm, symbol Connector:TestPoint
- added U2: TLV75533PDQNR, OpenRX-Shared:X2SON-4_L1.0-W1.0-P0.65-TL-EP, symbol OpenRX-Shared:TLV75533PDQNR
- added U3: SX1281IMLTRT, OpenRX-Shared:QFN-24_L4.0-W4.0-P0.50-TL-EP2.6, symbol OpenRX-Shared:SX1281IMLTRT
- added USB1: DEA102700LT-6307A2, OpenRX-Shared:FILTER-SMD_4P-L1.0-W0.5-L_DEA102700LT-XXX, symbol OpenRX-Shared:DEA102700LT-6307A2
Connections:
- net WIFI: now reaches U1.1 (LNA_IN)
- net WIFI: now also AE1.1 (ANT)
- net DIO1: now reaches U1.10 (MTDI)
- net DIO1: now also U3.8 (DIO1)
- net +3V3: now reaches U1.11 (VDD3P3_RTC)
- net +3V3: now also U1.17 (VDD3P3_CPU), U1.18 (VDD_SPI), U1.2 (VDD3P3), U1.3 (VDD3P3), U1.31 (VDDA), U1.32 (VDDA), C1.1, C10.1, C11.1, C13.1, C14.1, C15.1, C17.1, C19.1, C2.1, C3.1, C4.1, C5.1, OSC1.4 (VDD), R1.1, R2.1, R3.1, R4.1, U2.1 (OUT), U3.11 (VBAT_IO), U3.15 (VBAT), U3.2 (VDD_IN)
- net MISO: now reaches U1.12 (MTCK)
- net MISO: now also U3.16 (MISO_TX)
- net MOSI: now reaches U1.13 (MTDO)
- net MOSI: now also U3.17 (MOSI_RX)
- net NSS: now reaches U1.14 (GPIO8)
- net NSS: now also R2.2, U3.19 (NSS_CTS)
- net CHIP_BOOT: now reaches U1.15 (GPIO9)
- net CHIP_BOOT: now also R3.2
- net LED: now reaches U1.16 (GPIO10)
- net LED: now also D1.4 (DIN)
- net at U1.27 (U0RXD): now also TP1.1
- net at U1.28 (U0TXD): now also TP2.1
- net XTAL_N: now reaches U1.29 (XTAL_N)
- net XTAL_N: now also X1.3, C7.1
- net XTAL_P: now reaches U1.30 (XTAL_P)
- net XTAL_P: now also X1.1, C6.1
- net GND: now reaches U1.33 (EP)
- net GND: now also X1.2 (GND), X1.4 (GND), AE2.1, AE2.2, C1.2, C10.2, C11.2, C12.2, C13.2, C14.2, C15.2, C16.2, C17.2, C19.2, C2.2, C3.2, C4.2, C5.2, C6.2, C7.2, C8.2, C9.2, D1.3 (GND), OSC1.1 (GND), OSC1.2 (GND), TP4.1, U2.2 (GND), U2.5 (EP), U3.13 (GND), U3.20 (GND), U3.21 (GND), U3.23 (GND), U3.24 (GND), U3.25 (EP), U3.5 (GND), USB1.2 (GND), USB1.4 (GND)
- net RST: now reaches U1.6 (GPIO2)
- net RST: now also R4.2, U3.3 (NRESET)
- net CHIP_EN: now reaches U1.7 (CHIP_EN)
- net CHIP_EN: now also C8.1, R1.2
- net BUSY: now reaches U1.8 (GPIO3)
- net BUSY: now also U3.7 (BUSY)
- net SCK: now reaches U1.9 (MTMS)
- net SCK: now also U3.18 (SCK_RTSN)
- new net: U3.22 (RFIO), USB1.1 (IN)
- new net: AE2.3, USB1.3 (OUT)
- new net: C18.1, OSC1.3 (Out_Put)
- new net: C18.2, U3.4 (XTA)
- new net: C16.1, U3.1 (VR_PA)
- new net +5V: C12.1, C9.1, D1.2 (VDD), TP3.1, U2.3 (EN), U2.4 (IN)
- no-connect marks 0 -> 18
Other:
- note removed: "ANT1 2450AT18A100E L1/C16 Lite matching network No PA/LNA in the shared Lite core Keep antenna edge-placement and keepout in PCB work"
- note removed: "Firmware-critical mapping: GPIO4 = radio_sck GPIO5 = radio_dio1 GPIO6 = radio_miso GPIO7 = radio_mosi GPIO8 = radio_nss GPIO3 = radio_busy GPIO2 = radio_rst U0RXD = serial_rx U0TXD = serial_tx"
- note removed: "MCU + CLOCK"
- note removed: "OpenRX Shared SX1281 Receiver Core"
- note removed: "POWER"
- note removed: "RADIO + TCXO"
- note removed: "RF OUTPUT"
- note removed: "SX1281 pin contract already validated against local ExpressLRS: use logical radio_dio1 for IRQ, not radio_dio0. Keep BUSY and RST in the baseline."
- note removed: "This sheet is the reusable capture host for the Lite/Nano SX1281 family."
- note removed: "U1 ESP32-C3FH4 Y1 40MHz crystal R1/C6 EN RC delay R2 NSS pull-up R3 BOOT pull-up Optional GPIO9 boot pad Optional GPIO18/GPIO19 USB test pads"
- note removed: "U2 SX1281IMLTRT Y2 52MHz TCXO C9/C10/C12/C13 supply decoupling R5/C11 radio reset network LDO mode on VR_PA DIO2/DIO3 left unused in Lite baseline"
- note removed: "U3 TLV75533PDQNR C1 1uF local VIN cap C2 1uF local VOUT cap 10uF bulk at 5V entry 10uF bulk on +3.3V rail VIN 5V input rail VOUT +3.3V system rail"
- note removed: "Use the OpenRX-Shared library alias for imported symbols, footprints, and 3D models. Next capture pass on this sheet: place U3/U1/Y1/U2/Y2/ANT1, then add the passive network exactly from OpenRX-Lite/SCHEMATIC.md."
- moved on the sheet: AE1, X1

Commit message: Fix passive footprints to 0402/0603, add LCSC part numbers
- All caps/resistors: 0201 → 0402 (1005 Metric)
- 10uF bulk caps: 0402 → 0603 (1608 Metric)
- Added LCSC field to all 23 passives:
  100nF=C1525, 1uF=C52923, 10uF=C15525, 10pF=C32949,
  470nF=C1543, 1nF=C1523, 10k=C25744
- All JLCPCB basic parts, zero extended part setup fees on passives
Parts:
- C1, C13, C14, C15, C17, C2, C3, C4, C5: footprint Capacitor_SMD:C_0201_0603Metric -> Capacitor_SMD:C_0402_1005Metric; LCSC (none) -> C1525
- C10, C19, C8, C9: footprint Capacitor_SMD:C_0201_0603Metric -> Capacitor_SMD:C_0402_1005Metric; LCSC (none) -> C52923
- C11, C12: footprint Capacitor_SMD:C_0201_0603Metric -> Capacitor_SMD:C_0603_1608Metric; LCSC (none) -> C15525
- C16: footprint Capacitor_SMD:C_0201_0603Metric -> Capacitor_SMD:C_0402_1005Metric; LCSC (none) -> C1543
- C18: footprint Capacitor_SMD:C_0201_0603Metric -> Capacitor_SMD:C_0402_1005Metric; LCSC (none) -> C1523
- C6, C7: footprint Capacitor_SMD:C_0201_0603Metric -> Capacitor_SMD:C_0402_1005Metric; LCSC (none) -> C32949
- R1, R2, R3, R4: footprint Resistor_SMD:R_0201_0603Metric -> Resistor_SMD:R_0402_1005Metric; LCSC (none) -> C25744
