File: shared/sheets/esp32c3_sx1281_rx_core.kicad_sch (KiCad schematic)
At the start: 40 parts, among them U1 ESP32-C3FH4, U2 TLV75533PDQNR, U3 SX1281IMLTRT, U4 RFX2401C, X1 CJ17-400001010B20

Commit message: Fix Gemini crystal load caps to 18pF (C62164), matching Lite and Mono
Parts:
- C1, C13, C14, C15, C17, C2, C3, C4, C5: LCSC C14858 -> C76939
- C10, C19, C21, C8, C9: LCSC C77857 -> C76935
- C16: LCSC C304534 -> C85926
- C18: LCSC C80390 -> C66942
- C6, C7: LCSC C14854 -> C20069240
- R1, R2, R3, R4: LCSC C172043 -> C106225
Changed lines of the file:
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@@
 			)
 		)
-		(property "LCSC" "C77857"
+		(property "LCSC" "C76935"
 			(at 0 0 0)
 			(hide yes)
@@
 			)
 		)
-		(property "LCSC" "C77857"
+		(property "LCSC" "C76935"
 			(at 0 0 0)
 			(hide yes)
@@
 			)
 		)
-		(property "LCSC" "C14858"
+		(property "LCSC" "C76939"
 			(at 0 0 0)
 			(hide yes)
@@
 			)
 		)
-		(property "LCSC" "C77857"
+		(property "LCSC" "C76935"
 			(at 0 0 0)
 			(hide yes)
@@
 			)
 		)
-		(property "LCSC" "C172043"
+		(property "LCSC" "C106225"
 			(at 0 0 0)
 			(hide yes)
@@
 			)
 		)
-		(property "LCSC" "C14854"
+		(property "LCSC" "C20069240"
 			(at 0 0 0)
 			(hide yes)
@@
 			)
 		)
-		(property "LCSC" "C14858"
+		(property "LCSC" "C76939"
 			(at 0 0 0)
 			(hide yes)
@@
 			)
 		)
-		(property "LCSC" "C14854"
+		(property "LCSC" "C20069240"
 			(at 0 0 0)
 			(hide yes)
@@
 			)
 		)
-		(property "LCSC" "C14858"
+		(property "LCSC" "C76939"
 			(at 0 0 0)
 			(hide yes)
@@
 			)
 		)
-		(property "LCSC" "C80390"
+		(property "LCSC" "C66942"
 			(at 0 0 0)
 			(hide yes)
@@
 			)
 		)
-		(property "LCSC" "C172043"
+		(property "LCSC" "C106225"
 			(at 0 0 0)
 			(hide yes)
@@
 			)
 		)
-		(property "LCSC" "C172043"
+		(property "LCSC" "C106225"
 			(at 0 0 0)
 			(hide yes)
@@
 			)
 		)
-		(property "LCSC" "C77857"
+		(property "LCSC" "C76935"
 			(at 0 0 0)
 			(hide yes)
@@
 			)
 		)
-		(property "LCSC" "C172043"
+		(property "LCSC" "C106225"
 			(at 0 0 0)
 			(hide yes)
@@
 			)
 		)
-		(property "LCSC" "C14858"
+		(property "LCSC" "C76939"
 			(at 0 0 0)
 			(hide yes)
@@
 			)
 		)
-		(property "LCSC" "C14858"
+		(property "LCSC" "C76939"
 			(at 0 0 0)
 			(hide yes)
@@
 			)
 		)
-		(property "LCSC" "C14858"
+		(property "LCSC" "C76939"
 			(at 0 0 0)
 			(hide yes)
@@
 			)
 		)
-		(property "LCSC" "C304534"
+		(property "LCSC" "C85926"
 			(at 0 0 0)
 			(hide yes)
@@
 			)
 		)
-		(property "LCSC" "C77857"
+		(property "LCSC" "C76935"
 			(at 0 0 0)
 			(hide yes)
@@
 			)
 		)
-		(property "LCSC" "C14858"
+		(property "LCSC" "C76939"
 			(at 0 0 0)
 			(hide yes)
@@
 			)
 		)
-		(property "LCSC" "C14858"
+		(property "LCSC" "C76939"
 			(at 0 0 0)
 			(hide yes)
@@
 			)
 		)
-		(property "LCSC" "C14858"
+		(property "LCSC" "C76939"
 			(at 0 0 0)
 			(hide yes)
