File: OpenRX-Dual/OpenRX-Dual.kicad_sch (KiCad schematic)
At the start: 0 parts

Commit message: OpenRX-Dual: set up project, copy 900 schematic as base
Copy esp32c3_lr1121_900.kicad_sch as starting point.
Next step: add RFX2401C + DEA LPF + second UFL for 2.4GHz path in KiCad GUI.
Wire LR1121 RFIO_HF → DEA → RFX2401C, RFSW DIO5/DIO6 → RXEN/TXEN.
Other:
- added sheet ESP32-C3 + LR1121 Dual-Band (esp32c3_lr1121_dual.kicad_sch)
Changed lines of the file:
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@@
 (kicad_sch
-  (version 20231120)
-  (generator "eeschema")
-  (generator_version "9.0")
-  (paper "A3")
-  (symbol_instances)
+	(version 20260306)
+	(generator "eeschema")
+	(generator_version "10.0")
+	(paper "A3")
+	(sheet
+		(at 25.4 25.4)
+		(size 66.04 113.03)
+		(exclude_from_sim no)
+		(in_bom yes)
+		(on_board yes)
+		(dnp no)
+		(stroke
+			(width 0.1524)
+			(type solid)
+		)
+		(fill
+			(color 0 0 0 0)
+		)
+		(property "Sheetname" "ESP32-C3 + LR1121 Dual-Band"
+			(at 25.4 24.6888 0)
+			(show_name no)
+			(do_not_autoplace no)
+			(effects
+				(font
+					(size 1.27 1.27)
+				)
+				(justify left bottom)
+			)
+		)
+		(property "Sheetfile" "esp32c3_lr1121_dual.kicad_sch"
+			(at 25.4 141.478 0)
+			(show_name no)
+			(do_not_autoplace no)
+			(effects
+				(font
+					(size 1.27 1.27)
+				)
+				(justify left top)
+			)
+		)
+	)
+	(sheet_instances
+		(path "/"
+			(page "1")
+		)
+	)
+	(embedded_fonts no)
 )
