File: OpenRX-Gemini/OpenRX-Gemini.kicad_sch (KiCad schematic)
At the start: 0 parts

Commit message: OpenRX-Gemini: set up project, copy Dual schematic as base
Other:
- added sheet ESP32-C3 + 2x LR1121 Gemini (esp32c3_lr1121_gemini.kicad_sch)
Changed lines of the file:
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@@
 (kicad_sch
-  (version 20231120)
-  (generator "eeschema")
-  (generator_version "9.0")
-  (paper "A3")
-  (symbol_instances)
+	(version 20260306)
+	(generator "eeschema")
+	(generator_version "10.0")
+	(paper "A3")
+	(sheet
+		(at 25.4 25.4)
+		(size 66.04 113.03)
+		(exclude_from_sim no)
+		(in_bom yes)
+		(on_board yes)
+		(dnp no)
+		(stroke
+			(width 0.1524)
+			(type solid)
+		)
+		(fill
+			(color 0 0 0 0)
+		)
+		(property "Sheetname" "ESP32-C3 + 2x LR1121 Gemini"
+			(at 25.4 24.6888 0)
+			(show_name no)
+			(do_not_autoplace no)
+			(effects
+				(font
+					(size 1.27 1.27)
+				)
+				(justify left bottom)
+			)
+		)
+		(property "Sheetfile" "esp32c3_lr1121_gemini.kicad_sch"
+			(at 25.4 141.478 0)
+			(show_name no)
+			(do_not_autoplace no)
+			(effects
+				(font
+					(size 1.27 1.27)
+				)
+				(justify left top)
+			)
+		)
+	)
+	(sheet_instances
+		(path "/"
+			(page "1")
+		)
+	)
+	(embedded_fonts no)
 )
