File: OpenRX-Gemini/esp32c3_lr1121_gemini.kicad_sch (KiCad schematic)
At the start: 67 parts, among them T1 0900PC16J0042001E, T2 0900PC16J0042001E, U1 ESP32-C3FH4, U10 RFX2401C, U11 SKY13588-460LF, U2 TLV75533PDQNR, U3 TS2306A 240GF MSM 9_C2976675, U4 LR1121IMLTRT, U5 OW7EL89CENUYO3YLC-32M, U6 SKY13588-460LF, U7 RFX2401C, U8 OW7EL89CENUYO3YLC-32M, U9 LR1121IMLTRT, X1 CJ17-400001010B20

Commit message: Update schematics: Mono RF rewiring, SKY13414 port mapping, shared libs
Mono: disconnect IPD TX_LP (unused by ELRS), route TX_HP→RF3, RX→RF1,
RFX2401C ANT→RF4. Matches BetaFPV SuperX topology.

Co-Authored-By: Claude Opus 4.6 (1M context) <noreply@anthropic.com>
Parts:
- removed C14: 1uF, Capacitor_SMD:C_0201_0603Metric, symbol Device:C
- removed C15: 220pF, Capacitor_SMD:C_0201_0603Metric, symbol Device:C
- removed C16: 0.3pF, Capacitor_SMD:C_0201_0603Metric, symbol Device:C
- removed C17: 10pF, Capacitor_SMD:C_0201_0603Metric, symbol Device:C
- removed C20: 4.7uF, Capacitor_SMD:C_0402_1005Metric, symbol Device:C
- removed C22: 100nF, Capacitor_SMD:C_0201_0603Metric, symbol Device:C
- removed L1: 10uH, Inductor_SMD:L_0603_1608Metric, symbol Device:L
- removed R6, R7: 220R, Resistor_SMD:R_0201_0603Metric, symbol Device:R
- removed U11, U6: SKY13588-460LF, OpenRX-Shared:QFN-12_L2.0-W2.0-P0.50-BL-EP0.8, symbol OpenRX-Shared:SKY13588-460LF
- removed U4: LR1121IMLTRT, OpenRX-Shared:QFN-32_L5.0-W5.0-P0.50-BL-EP3.7, symbol OpenRX-Shared:LR1121IMLTRT
- removed U5: OW7EL89CENUYO3YLC-32M, OpenRX-Shared:OSC-SMD_4P-L2.0-W1.6-BL_TXC_7Z, symbol OpenRX-Shared:OW7EL89CENUYO3YLC-32M
- removed U7: RFX2401C, OpenRX-Shared:QFN-16_L3.0-W3.0-P0.50-BL-EP1.7, symbol OpenRX-Shared:RFX2401C
- removed USB3: DEA102700LT-6307A2, OpenRX-Shared:FILTER-SMD_4P-L1.0-W0.5-L_DEA102700LT-XXX, symbol OpenRX-Shared:DEA102700LT-6307A2
- added C19: 0.3pF, Capacitor_SMD:C_0201_0603Metric, symbol Device:C
- added C3, C5, C7: 100nF, Capacitor_SMD:C_0201_0603Metric, symbol Device:C
- added C8: 10pF, Capacitor_SMD:C_0201_0603Metric, symbol Device:C
- added C9: 4.7uF, Capacitor_SMD:C_0402_1005Metric, symbol Device:C
- added L2: 10uH, Inductor_SMD:L_0603_1608Metric, symbol Device:L
- added R3, R8: 220R, Resistor_SMD:R_0201_0603Metric, symbol Device:R
- added U1: OW7EL89CENUYO3YLC-32M, OpenRX-Shared:OSC-SMD_4P-L2.0-W1.6-BL_TXC_7Z, symbol OpenRX-Shared:OW7EL89CENUYO3YLC-32M
- added U11, U7: SKY13414-485LF, OpenRX-Shared:QFN-14_L2.0-W2.0-P0.45-BL-EP, symbol OpenRX-Shared:SKY13414-485LF
- added U2: LR1121IMLTRT, OpenRX-Shared:QFN-32_L5.0-W5.0-P0.50-BL-EP3.7, symbol OpenRX-Shared:LR1121IMLTRT
- added U5: RFX2401C, OpenRX-Shared:QFN-16_L3.0-W3.0-P0.50-BL-EP1.7, symbol OpenRX-Shared:RFX2401C
- added USB1: 2450FM07D0034, OpenRX-Shared:FILTER-SMD_4P-L1.0-W0.5-L_DEA102700LT-XXX, symbol OpenRX-Shared:DEA102700LT-6307A2
- C13: value 10pF -> 100nF; LCSC C20069240 -> C76939
- C21: value 100nF -> 220pF; LCSC C76939 -> C62548
- C23: value 100nF -> 1uF; LCSC C76939 -> C76935
- C27: value 100nF -> 10pF; LCSC C76939 -> C20069240
- USB2: value DEA102700LT-6307A2 -> 2450FM07D0034; LCSC C574024 -> C2651081; LCSC Part C574024 -> (none)
- renumbered C6 to C1, C1 to C10, C2 to C11, C18 to C12, C12 to C14, C3 to C15, C9 to C16, C4 to C17, C5 to C18, C8 to C2, C10 to C20, C11 to C22, C7 to C4, C19 to C6, L2 to L1, R4 to R2, R5 to R4, R8 to R5, R2 to R6, R3 to R7, U1 to U3, U3 to U4, U2 to U6
Connections:
- net +3V3: now also C13.2, C23.1, C24.1, C3.1, L2.2, U11.4 (VDD), U2.15 (VBAT), U2.2 (VBAT_RF), U5.14 (VDD), U5.16 (VDD), U7.4 (VDD); no longer C24.2, C25.1
- net BUSY2: now also U2.25 (DIO0/BUSY)
- net DIO7-1: now also U11.5 (V3)
- net DIO7-2: now also U2.11 (DIO7), U7.5 (V3)
- net DIO8-1: now also U11.6 (V2)
- net DIO8-2: now also U2.10 (DIO8), U7.6 (V2)
- net GND: now also C13.1, C23.2, C24.2, C25.1, C19.2, C3.2, C5.1, C7.1, C9.2, U1.1 (GND), U1.2 (GND), U11.15 (EP), U11.7 (V1), U2.13 (GND), U2.33 (EP), U5.1 (GND), U5.11 (GND), U5.12 (GND), U5.15 (GND), U5.17 (EP), U5.2 (GND), U5.3 (GND), U5.7 (GND), U5.8 (GND), U5.9 (GND), U7.15 (EP), U7.7 (V1), USB1.2 (GND), USB1.4 (GND); no longer C23.1, C24.1, C25.2, C27.1
- net IRQ2: now also U2.9 (DIO9)
- net MISO: now also U2.21 (DIO4)
- net MOSI: now also U2.22 (DIO3)
- net NSS2: now also U2.24 (DIO1)
- net RST2: now also U2.6 (NRESET)
- net RXEN2: now also U2.20 (DIO5), U5.6 (RXEN)
- net SCK: now also U2.23 (DIO2)
- net TXEN2: now also U2.19 (DIO6), U5.5 (TXEN)
- net at C30.1, U10.10 (ANT): now also U11.2 (RF3)
- net at JP1.1 (SIG): now also U7.13 (ANT)
- net at U8.4 (VDD), U9.3 (VTCXO): now also C25.2; no longer C26.2
- net at USB2.1 (IN): now also U9.26 (RFIO_HF)
- net at T1.4 (RFI_N_LFO): now also U2.29 (RFI_N_LF0)
- net at T1.3 (RFI_P_LFO): now also U2.30 (RFI_P_LF0)
- net at T1.2 (RFO_LP_LF): now also U2.31 (RFO_LP_LF)
- net at T1.1 (RFO_HP_LF): now also U2.32 (RFO_HP_LF)
- net at U8.3 (OUTPUT): now also R8.2
- net at U9.4 (XTA): now also C27.2
- net at JP2.1 (SIG): now also U11.13 (ANT)
- net at U9.12 (VREG): now also C26.2; no longer C27.2
- net at U10.4 (TXRX): now also USB2.3 (OUT)
- new net: C5.2, U1.4 (VDD), U2.3 (VTCXO)
- new net: C9.1, U2.1 (VR_PA)
- new net: R3.2, U1.3 (OUTPUT)
- new net: U2.26 (RFIO_HF), USB1.1 (IN)
- new net: U5.4 (TXRX), USB1.3 (OUT)
- new net: C8.1, R3.1
- new net: C8.2, U2.4 (XTA)
- new net: C27.1, R8.1
- new net: C19.1, U5.10 (ANT), U7.2 (RF3)
- new net: T1.6 (RX), U7.3 (RF1)
- new net: T1.8 (TX_LP), U7.10 (RF4)
- new net: T1.9 (TX_HP), U7.9 (RF2)
- new net: T2.6 (RX), U11.3 (RF1)
- new net: T2.8 (TX_LP), U11.10 (RF4)
- new net: T2.9 (TX_HP), U11.9 (RF2)
- new net: L2.1, U2.14 (DCC_SW)
- new net: C7.2, U2.12 (VREG)
- no-connect marks 28 -> 26
