File: OpenRX-Mono/OpenRX-Mono.kicad_pcb (KiCad board)
At the start: 4 copper layers, 9.6 x 13.6 mm, 47 parts, among them T1 0900PC16J0042001E, U1 ESP32-C3FH4, U2 TLV75533PDQNR, U3 TS2306A 240GF MSM 9_C2976675, U4 LR1121IMLTRT, U5 OW7EL89CENUYO3YLC-32M, U6 SKY13588-460LF, U7 RFX2401C, X1 CJ17-400001010B20

Commit message: Repo cleanup: final state for handoff
- Clean README with architecture, BOM, CE notes, status
- Remove dated analysis files (absorbed into FINAL_NETLIST + KICAD_WORKFLOW)
- Remove stale OpenRX-Dual (archived), ERC reports, backups, prl files
- Updated .gitignore for .kicad_dru, production backups
- CERN-OHL-S v2 license confirmed
- 3 active projects: Lite, Mono, Gemini
- Schematics final, initial PCB layouts done, routing in progress
Other:
- copper layers 4 -> 6
Changed lines of the file:
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@@
 	(generator_version "10.0")
 	(general
-		(thickness 1.0278)
+		(thickness 1.0)
 		(legacy_teardrops no)
 	)
@@
 		(4 "In1.Cu" signal)
 		(6 "In2.Cu" signal)
+		(8 "In3.Cu" signal)
+		(10 "In4.Cu" signal)
 		(2 "B.Cu" signal)
 		(9 "F.Adhes" user "F.Adhesive")
@@
 			(layer "dielectric 2"
 				(type "core")
-				(thickness 0.7074)
+				(thickness 0.16)
 				(material "FR4")
 				(epsilon_r 4.5)
@@
 			(layer "dielectric 3"
 				(type "prepreg")
+				(thickness 0.3292)
+				(material "FR4")
+				(epsilon_r 4.5)
+				(loss_tangent 0.02)
+			)
+			(layer "In3.Cu"
+				(type "copper")
+				(thickness 0.0152)
+			)
+			(layer "dielectric 4"
+				(type "core")
+				(thickness 0.16)
+				(material "FR4")
+				(epsilon_r 4.5)
+				(loss_tangent 0.02)
+			)
+			(layer "In4.Cu"
+				(type "copper")
+				(thickness 0.0152)
+			)
+			(layer "dielectric 5"
+				(type "prepreg")
 				(thickness 0.1)
