File: OpenRX-Mono/esp32c3_lr1121_mono.kicad_sch (KiCad schematic)
At the start: 47 parts, among them T1 0900PC16J0042001E, U1 ESP32-C3FH4, U2 TLV75533PDQNR, U3 TS2306A 240GF MSM 9_C2976675, U4 LR1121IMLTRT, U5 OW7EL89CENUYO3YLC-32M, U6 SKY13588-460LF, U7 RFX2401C, X1 CJ17-400001010B20

Commit message: Repo cleanup: final state for handoff
- Clean README with architecture, BOM, CE notes, status
- Remove dated analysis files (absorbed into FINAL_NETLIST + KICAD_WORKFLOW)
- Remove stale OpenRX-Dual (archived), ERC reports, backups, prl files
- Updated .gitignore for .kicad_dru, production backups
- CERN-OHL-S v2 license confirmed
- 3 active projects: Lite, Mono, Gemini
- Schematics final, initial PCB layouts done, routing in progress
Parts:
- C16: LCSC (none) -> C76927
Changed lines of the file:
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@@
 			)
 		)
-		(property "LCSC" ""
+		(property "LCSC" "C76927"
 			(at 414.02 299.72 0)
 			(hide yes)
