File: OpenRX-Mono/esp32c3_lr1121_mono.kicad_sch (KiCad schematic)
At the start: 47 parts, among them T1 0900PC16J0042001E, U1 ESP32-C3FH4, U2 TLV75533PDQNR, U3 TS2306A 240GF MSM 9_C2976675, U4 LR1121IMLTRT, U5 OW7EL89CENUYO3YLC-32M, U6 SKY13588-460LF, U7 RFX2401C, X1 CJ17-400001010B20

Commit message: Update schematics: Mono RF rewiring, SKY13414 port mapping, shared libs
Mono: disconnect IPD TX_LP (unused by ELRS), route TX_HP→RF3, RX→RF1,
RFX2401C ANT→RF4. Matches BetaFPV SuperX topology.

Co-Authored-By: Claude Opus 4.6 (1M context) <noreply@anthropic.com>
Parts:
- removed U6: SKY13588-460LF, OpenRX-Shared:QFN-12_L2.0-W2.0-P0.50-BL-EP0.8, symbol OpenRX-Shared:SKY13588-460LF
- removed USB2: DEA102700LT-6307A2, OpenRX-Shared:FILTER-SMD_4P-L1.0-W0.5-L_DEA102700LT-XXX, symbol OpenRX-Shared:DEA102700LT-6307A2
- added FL1: 2450FM07D0034T, OpenRX-Shared:FILTER-SMD_4P-L1.0-W0.5-L, symbol OpenRX-Shared:2450FM07D0034T
- added U8: SKY13414-485LF, OpenRX-Shared:QFN-14_L2.0-W2.0-P0.45-BL-EP, symbol OpenRX-Shared:SKY13414-485LF
Connections:
- net +3V3: now also U8.4 (VDD)
- net DIO7-1: now also U8.5 (V3)
- net DIO8-1: now also U8.6 (V2)
- net GND: now also FL1.2 (GND), FL1.4 (GND), U8.15 (EP), U8.7 (V1)
- net at C16.1, U7.10 (ANT): now also U8.10 (RF4)
- net at JP1.1 (SIG): now also U8.13 (ANT)
- net at U4.26 (RFIO_HF): now also FL1.1 (IN)
- net at U7.4 (TXRX): now also FL1.3 (OUT)
- new net: T1.9 (TX_HP), U8.2 (RF3)
- new net: T1.6 (RX), U8.3 (RF1)
- now unconnected: T1.8 (TX_LP)
- no-connect marks 22 -> 28
Other:
- moved on the sheet: JP1
