File: OpenRX-Mono/esp32c3_lr1121_mono.kicad_sch (KiCad schematic)
At the start: 47 parts, among them T1 0900PC16J0042001E, U1 ESP32-C3FH4, U2 TLV75533PDQNR, U3 TS2306A 240GF MSM 9_C2976675, U4 LR1121IMLTRT, U5 OW7EL89CENUYO3YLC-32M, U7 RFX2401C, U8 SKY13414-485LF, X1 CJ17-400001010B20

Commit message: initial routing for all
Parts:
- removed C10: 1uF, Capacitor_SMD:C_0201_0603Metric, symbol Device:C
- added R5: 10k, Resistor_SMD:R_0201_0603Metric, symbol Device:R
- added TP5: Boot, OpenRX-Shared:SolderPad_1.2x2.0mm, symbol Connector:TestPoint
- C1, C18, C2, C21, C22, C23, C24, C3, C4, C5: LCSC Part (none) -> C76939
- C11, C12: LCSC Part (none) -> C15525
- C13: LCSC C20069240 -> C76921; LCSC Part (none) -> C76921
- C14, C19, C8, C9: LCSC Part (none) -> C76935
- C15: LCSC Part (none) -> C62548
- C16: LCSC Part (none) -> C76927
- C20: LCSC Part (none) -> C23733
- C6, C7: LCSC Part (none) -> C62164
- L1: LCSC C6808014 -> C1035; LCSC Part (none) -> C1035
- L2: LCSC Part (none) -> C206441
- R1, R2, R3, R4: LCSC Part (none) -> C106225
- R6: LCSC Part (none) -> C274342
Connections:
- net +3V3: now also R5.1
- net BUTTON: now also TP5.1
- net LED: now also R5.2
