File: OpenRX-Lite-UFL/esp32c3_sx1281_lite.kicad_sch (KiCad schematic)
At the start: 39 parts, among them U1 ESP32-C3FH4, U2 TLV75533PDQNR, U3 SX1281IMLTRT, X1 CJ17-400001010B20

Commit message: initial routing for all
Parts:
- C1, C3: LCSC Part (none) -> C62164
- C10, C15, C2, C4: LCSC Part (none) -> C76935
- C11, C12, C13, C14, C17, C18, C5, C6, C7, C9: LCSC Part (none) -> C76939
- C16, C8: LCSC Part (none) -> C15525
- C19: LCSC Part (none) -> C66942
- C20: LCSC Part (none) -> C85926
- L1: LCSC Part (none) -> C206441
- R1, R2, R3, R4: LCSC Part (none) -> C106225
