File: OpenRX-Lite-UFL/OpenRX-Lite-UFL.kicad_pcb (KiCad board)
At the start: 6 copper layers, 8.2 x 12.2 mm, 39 parts, among them U1 ESP32-C3FH4, U2 TLV75533PDQNR, U3 SX1281IMLTRT, X1 CJ17-400001010B20

Commit message: initial routing for all
Parts:
- moved C14 0.57 mm to (180.8, 96.1)
- moved C20 0.36 mm to (180.8, 95.6)
- moved OSC1 0.25 mm to (180.4, 98.8)
- moved C13 0.22 mm to (181.8, 99.4)
- moved C19 0.16 mm to (180.8, 97.2)
Routing:
- net GND: track 39.0 -> 45.8 mm, vias 23 -> 29
- net +3V3: track 19.8 -> 21.5 mm
- net unconnected-(AE1-Pad2): vias 0 -> 1

Commit message: final route
Parts:
- FL1: value 2450FM07D0034 -> 2450FM07D0034T; footprint OpenRX-Shared:FILTER-SMD_4P-L1.0-W0.5-L_DEA102700LT-XXX -> OpenRX-Shared:FILTER-SMD_4P-L1.0-W0.5-L
- moved TP1 2.20 mm to (180.0, 101.7)
- moved TP2 2.20 mm to (182.2, 101.7)
- moved FL1 0.09 mm to (183.2, 94.0)
Routing:
- net Net-(U1-U0RXD): track 10.7 -> 11.0 mm, vias 3 -> 2
- net Net-(U1-U0TXD): track 9.84 -> 9.68 mm, vias 2 -> 1
Other:
- board size 8.2 x 12.2 mm -> 8.5 x 12.3 mm
